Commit message: start work on simulating arm and head of robot

File: ros_ws/src/bearmax_description/urdf/robot_base.xacro (robot description, xacro)
@@ -33,16 +33,17 @@
     <link name="body">
         <visual>
-            <origin xyz="0 0 0.05"/>
+            <origin xyz="0 0 0.15"/>
             <geometry>
-                <cylinder radius="0.2" length="0.2"/>
+                <cylinder radius="0.2" length="0.4"/>
             </geometry>
             <material name="blue"/>
         </visual>
         <collision>
-            <origin xyz="0 0 0.05"/>
+            <origin xyz="0 0 0.15"/>
             <geometry>
-                <cylinder radius="0.2" length="0.2"/>
+                <cylinder radius="0.2" length="0.4"/>
             </geometry>
         </collision>
     </link>
+    <xacro:include filename="arm.xacro" />
 </robot>
