Commit message: Add head to description

File: ros_ws/src/bearmax_description/urdf/bearmax_description.urdf (robot description, URDF)
Before this commit: robot None, 16 links, 15 joints
Links:
- removed link camera_optical_link
Joints:
- removed joint camera_optical_joint
- joint chassis_joint: limit lower=-${pi/2} upper=${pi/2} effort=10 velocity=100 -> lower=-1.57 upper=1.57 effort=10 velocity=100
- joint left_arm_elbow_joint: limit lower=-${pi/2} upper=${pi/2} effort=10 velocity=100 -> lower=-1.57 upper=1.57 effort=10 velocity=100
- joint left_arm_rotator_joint: limit lower=-${pi/2} upper=${pi/2} effort=10 velocity=100 -> lower=-1.57 upper=1.57 effort=10 velocity=100
- joint left_arm_shoulder_joint: limit lower=-${pi/2} upper=${pi/2} effort=10 velocity=100 -> lower=-1.57 upper=1.57 effort=10 velocity=100
- joint left_ear_pitch_joint: limit lower=-${pi/2} upper=${pi/2} effort=10 velocity=100 -> lower=-1.57 upper=1.57 effort=10 velocity=100
- joint left_ear_rotator_joint: limit lower=-${pi/2} upper=${pi/2} effort=10 velocity=100 -> lower=-1.57 upper=1.57 effort=10 velocity=100
- joint right_arm_elbow_joint: limit lower=-${pi/2} upper=${pi/2} effort=10 velocity=100 -> lower=-1.57 upper=1.57 effort=10 velocity=100
- joint right_arm_rotator_joint: limit lower=-${pi/2} upper=${pi/2} effort=10 velocity=100 -> lower=-1.57 upper=1.57 effort=10 velocity=100
- joint right_arm_shoulder_joint: limit lower=-${pi/2} upper=${pi/2} effort=10 velocity=100 -> lower=-1.57 upper=1.57 effort=10 velocity=100
- joint right_ear_pitch_joint: limit lower=-${pi/2} upper=${pi/2} effort=10 velocity=100 -> lower=-1.57 upper=1.57 effort=10 velocity=100
- joint right_ear_rotator_joint: limit lower=-${pi/2} upper=${pi/2} effort=10 velocity=100 -> lower=-1.57 upper=1.57 effort=10 velocity=100
