Commit message: Finished urdf simulation

File: ros_ws/src/bearmax_description/urdf/bearmax_description.urdf.xacro (robot description, xacro)
@@ -3,5 +3,5 @@
   <link
     name="base_link">
-    <inertial>
+    <!--<inertial>
       <origin
         xyz="-0.17187 0.041344 0.40096"
@@ -16,5 +16,5 @@
         iyz="-2.4791E-06"
         izz="0.0003814" />
-    </inertial>
+    </inertial>-->
     <visual>
       <origin
@@ -86,5 +86,5 @@
     <origin
       xyz="-0.17961 -0.40208 0.012"
-      rpy="1.5708 0 1.5708" />
+      rpy="1.5708 0 ${pi/2}" />
     <parent
       link="base_link" />
@@ -104,5 +104,5 @@
       <origin
         xyz="-0.032811 0.026124 -0.043368"
-        rpy="0 0 0" />
+        rpy="${pi} 0 0" />
       <mass
         value="2.6697" />
@@ -118,5 +118,5 @@
       <origin
         xyz="0 0 0"
-        rpy="0 0 0" />
+          rpy="${pi} 0 0" />
       <geometry>
         <mesh
@@ -132,5 +132,5 @@
       <origin
         xyz="0 0 0"
-        rpy="0 0 0" />
+          rpy="${pi} 0 0" />
       <geometry>
         <mesh
@@ -144,5 +144,5 @@
     <origin
       xyz="0 0.4005 0"
-      rpy="3.1416 -1.5708 0" />
+      rpy="3.1416 -${pi/2} 0" />
     <parent
       link="chassis_link" />
@@ -174,5 +174,5 @@
       <geometry>
         <mesh
-          filename="package://bearmax_description/meshes/left_arm_shoulder_link.STL" />
+          filename="package://bearmax_description/meshes/left_arm_shoulder_link01.STL" />
       </geometry>
       <material
@@ -188,5 +188,5 @@
       <geometry>
         <mesh
-          filename="package://bearmax_description/meshes/left_arm_shoulder_link.STL" />
+          filename="package://bearmax_description/meshes/left_arm_shoulder_link01.STL" />
       </geometry>
     </collision>
@@ -196,6 +196,10 @@
     type="revolute">
     <origin
+        xyz="0.14497 -0.027824 0.0102"
+        rpy="${pi/2} ${3*pi/4} 1.3963"
+    />
+    <!--origin
       xyz="0.1153 0.022388 -0.010325"
-      rpy="3.1416 -0.080918 -1.3963" />
+      rpy="3.1416 -0.080918 -1.3963" /-->
     <parent
       link="torso_link" />
@@ -203,5 +207,5 @@
       link="left_arm_shoulder_link" />
     <axis
-      xyz="0 1 0" />
+      xyz="0 0 1" />
     <limit
       lower="-${pi/2}"
@@ -228,6 +232,7 @@
     <visual>
       <origin
-        xyz="0 0 0"
-        rpy="0 0 0" />
+          xyz="0.0575 0.0325 -0.02125"
+          rpy="0 ${pi} ${pi}"
+      />
       <geometry>
         <mesh
@@ -242,6 +247,7 @@
     <collision>
       <origin
-        xyz="0 0 0"
-        rpy="0 0 0" />
+          xyz="0.0575 0.0325 -0.02125"
+          rpy="0 ${pi} ${pi}"
+      />
       <geometry>
         <mesh
@@ -254,6 +260,10 @@
     type="revolute">
     <origin
-      xyz="0 0.01 0"
-      rpy="3.1416 -0.54847 1.5708" />
+        xyz="0.012 0.0319 0.019941"
+        rpy="0 0.86598 ${pi}"
+    />
+    <!--origin
+      xyz="0.012 -0.0319 -0.019941"
+      rpy="0 -0.54847 ${pi/2}" /-->
     <parent
       link="left_arm_shoulder_link" />
@@ -286,5 +296,5 @@
     <visual>
       <origin
-        xyz="0 0 0"
+        xyz="-0.13325 0.035 -0.05875"
         rpy="0 0 0" />
       <geometry>
@@ -300,5 +310,5 @@
     <collision>
       <origin
-        xyz="0 0 0"
+        xyz="-0.13325 0.035 -0.05875"
         rpy="0 0 0" />
       <geometry>
@@ -312,6 +322,10 @@
     type="revolute">
     <origin
+        xyz="-0.0018031 -0.112 0.0018031"
+        rpy="${pi+2.1424} 0.57212 -2.2705"
+    />
+    <!--origin
       xyz="-0.020548 0 -0.012555"
-      rpy="2.2751 -0.38212 1.9844" />
+      rpy="2.2751 -0.38212 1.9844" /-->
     <parent
       link="left_arm_rotator_link" />
@@ -370,6 +384,10 @@
     type="revolute">
     <origin
+        xyz="-0.14497 -0.027824 0.0102"
+        rpy="-${pi/2} ${pi/4} -1.3963"
+    />
+    <!--origin
       xyz="-0.14497 0.027824 -0.0102"
-      rpy="1.5708 -1.5367 1.3963" />
+      rpy="1.5708 -1.5367 1.3963" /-->
     <parent
       link="torso_link" />
@@ -377,5 +395,5 @@
       link="right_arm_shoulder_link" />
     <axis
-      xyz="0 1 0" />
+      xyz="0 0 1" />
     <limit
       lower="-${pi/2}"
@@ -429,5 +447,5 @@
     <origin
       xyz="0.012 0.0319 -0.019941"
-      rpy="0 0.86598 3.1416" />
+        rpy="0 0.86598 ${pi}" />
     <parent
       link="right_arm_shoulder_link" />
@@ -517,7 +535,4 @@
     </inertial>
     <visual>
-      <origin
-        xyz="0 0 0"
-        rpy="0 0 0" />
       <geometry>
         <mesh
@@ -531,7 +546,4 @@
     </visual>
     <collision>
-      <origin
-        xyz="0 0 0"
-        rpy="0 0 0" />
       <geometry>
         <mesh
@@ -542,14 +554,12 @@
   <joint
     name="head_platform_joint"
-    type="fixed">
-    <origin
-      xyz="0 0.074456 0"
-      rpy="3.1416 0 3.1416" />
+    type="floating">
+    <origin
+      xyz="0 -0.074456 0"
+      rpy="0 0 ${pi}" />
     <parent
       link="torso_link" />
     <child
       link="head_platform_link" />
-    <axis
-      xyz="0 0 0" />
   </joint>
   <link
@@ -571,6 +581,7 @@
     <visual>
       <origin
-        xyz="0 0 0"
-        rpy="0 0 0" />
+          xyz="-0.0225 -0.01003 0"
+          rpy="0 0 0"
+      />
       <geometry>
         <mesh
@@ -585,5 +596,5 @@
     <collision>
       <origin
-        xyz="0 0 0"
+        xyz="-0.0225 -0.01003 0"
         rpy="0 0 0" />
       <geometry>
@@ -596,7 +607,12 @@
     name="left_ear_rotator_joint"
     type="revolute">
-    <origin
-      xyz="-0.068776 0.11753 -0.0008258"
-      rpy="-0.00010149 -0.0069114 -1.0472" />
+    <!--origin
+        xyz="-0.068776 0.11753 -0.0008258"
+        rpy="-0.00010149 -0.0069114 -1.0472"
+    /-->
+    <origin
+        xyz="-0.048776 0.1025 -0.0008258"
+        rpy="-0.00010149 -0.0069114 -1.0472"
+    />
     <parent
       link="head_platform_link" />
@@ -604,5 +620,5 @@
       link="left_ear_rotator_link" />
     <axis
-      xyz="0 1 0" />
+      xyz="1 0 0" />
     <limit
       lower="-${pi/2}"
@@ -655,6 +671,6 @@
     type="revolute">
     <origin
-      xyz="-0.005175 0.0299 0"
-      rpy="-3.1416 -0.0069114 3.1416" />
+      xyz="-0.0287 0.01955 0"
+      rpy="-${pi} -0.0069114 ${pi}" />
     <parent
       link="left_ear_rotator_link" />
@@ -772,5 +788,5 @@
     <origin
       xyz="0.01955 0.0287 0"
-      rpy="-3.1416 -0.0069114 1.5708" />
+      rpy="-${pi} -0.0069114 ${pi/2}" />
     <parent
       link="right_ear_rotator_link" />
@@ -830,5 +846,5 @@
     <origin
       xyz="0.0007478 0.0791 -0.054095"
-      rpy="-1.5708 0.013823 3.1416" />
+      rpy="-${pi/2} 0.013823 ${pi}" />
     <parent
       link="head_platform_link" />

Commit message: Implement initially working ros2 control hardware interface and controllers

File: ros_ws/src/bearmax_description/urdf/bearmax_description.urdf.xacro (robot description, xacro)
@@ -3,7 +3,7 @@
   <link
     name="base_link">
-    <!--<inertial>
-      <origin
-        xyz="-0.17187 0.041344 0.40096"
+    <inertial>
+      <origin
+        xyz="-0.17187 -0.4 0.051344"
         rpy="0 0 0" />
       <mass
@@ -16,6 +16,35 @@
         iyz="-2.4791E-06"
         izz="0.0003814" />
-    </inertial>-->
-    <visual>
+    </inertial>
+    <visual>
+      <origin
+        xyz="0 0 0"
+        rpy="0 0 0" />
+      <geometry>
+        <mesh
+            filename="package://bearmax_description/meshes/base_link.STL"
+        />
+      </geometry>
+      <!--material
+        name="">
+        <color
+          rgba="0.79216 0.81961 0.93333 1" />
+      </material-->
+    </visual>
+    <!--visual>
+      <origin
+          xyz="-0.17961 -0.40208 -0.01"
+          rpy="0 0 0"
+      />
+      <geometry>
+          <box size="0.3 0.3 0.01"/>
+      </geometry>
+      <material
+        name="black">
+        <color
+          rgba="0 0 0 1" />
+      </material>
+    </visual-->
+    <collision>
       <origin
         xyz="0 0 0"
@@ -25,17 +54,13 @@
           filename="package://bearmax_description/meshes/base_link.STL" />
       </geometry>
-      <material
-        name="">
-        <color
-          rgba="0.79216 0.81961 0.93333 1" />
-      </material>
-    </visual>
-    <collision>
-      <origin
-        xyz="0 0 0"
-        rpy="0 0 0" />
-      <geometry>
-        <mesh
-          filename="package://bearmax_description/meshes/base_link.STL" />
+    </collision>
+    <!-- To prevent the robot from tipping over cause of bad interals -->
+    <collision>
+      <origin
+          xyz="-0.17961 -0.40208 -0.01"
+          rpy="0 0 0"
+      />
+      <geometry>
+          <box size="0.3 0.3 0.01"/>
       </geometry>
     </collision>
@@ -552,14 +577,51 @@
     </collision>
   </link>
-  <joint
-    name="head_platform_joint"
-    type="floating">
-    <origin
-      xyz="0 -0.074456 0"
-      rpy="0 0 ${pi}" />
-    <parent
-      link="torso_link" />
-    <child
-      link="head_platform_link" />
+  <!-- Head Platform Joints -->
+  <joint name="head_platform_pitch_joint" type="revolute">
+    <origin
+        xyz="0 -0.074456 0"
+        rpy="0 0 ${pi}"
+    />
+    <parent link="torso_link" />
+    <child link="head_platform_roll_link" />
+    <limit
+        lower="-${pi/6}"
+        upper="${pi/6}"
+        effort="10"
+        velocity="100"
+    />
+    <axis xyz="1 0 0" />
+  </joint>
+  <link name="head_platform_roll_link"></link>
+  <joint name="head_platform_roll_joint" type="revolute">
+    <origin
+        xyz="0 0 0"
+        rpy="0 0 0"
+    />
+    <parent link="head_platform_roll_link" />
+    <child link="head_platform_yaw_link" />
+    <limit
+        lower="-${pi/6}"
+        upper="${pi/6}"
+        effort="10"
+        velocity="100"
+    />
+    <axis xyz="0 0 1" />
+  </joint>
+  <link name="head_platform_yaw_link"></link>
+  <joint name="head_platform_yaw_joint" type="revolute">
+    <origin
+        xyz="0 0 0"
+        rpy="0 0 0"
+    />
+    <parent link="head_platform_yaw_link" />
+    <child link="head_platform_link" />
+    <limit
+        lower="-${pi/2}"
+        upper="${pi/2}"
+        effort="10"
+        velocity="100"
+    />
+    <axis xyz="0 1 0" />
   </joint>
   <link

File: ros_ws/src/bearmax_description/urdf/hardware.ros2_control.xacro (robot description, xacro)
@@ -1,3 +1,3 @@
-<?xml version="1.0"?>
+<?xml version="180.0"?>
 <robot xmlns:xacro="http://www.ros.org/wiki/xacro">
     <xacro:unless value="$(arg sim_mode)">
@@ -5,7 +5,7 @@
             <hardware>
                 <plugin>bearmax_hardware/BearmaxArduino</plugin>
-                <param name="device">/dev/ttyUSB0</param>
+                <param name="device">/dev/ttyACM0</param>
                 <param name="baud_rate">57600</param>
-                <param name="timeout">1000</param>
+                <param name="timeout">180000</param>
             </hardware>
             <!-- Chassis Joints -->
@@ -18,7 +18,6 @@
             </joint>
             <!-- Head Joints -->
-            <!-- TODO: Determine if can compute servo positions on ros -->
-            <!--
-            <joint name="left_ear_rotation">
+            <!-- Head Platform -->
+            <joint name="head_platform_roll_joint">
                 <command_interface name="position">
                     <param name="min">0</param>
@@ -27,5 +26,5 @@
                 <state_interface name="position" />
             </joint>
-            <joint name="left_ear_pitch">
+            <joint name="head_platform_pitch_joint">
                 <command_interface name="position">
                     <param name="min">0</param>
@@ -34,5 +33,27 @@
                 <state_interface name="position" />
             </joint>
-            <joint name="right_ear_rotation">
+            <joint name="head_platform_yaw_joint">
+                <command_interface name="position">
+                    <param name="min">0</param>
+                    <param name="max">180</param>
+                </command_interface>
+                <state_interface name="position" />
+            </joint>
+            <!-- Ears -->
+            <joint name="left_ear_rotator_joint">
+                <command_interface name="position">
+                    <param name="min">0</param>
+                    <param name="max">180</param>
+                </command_interface>
+                <state_interface name="position" />
+            </joint>
+            <joint name="left_ear_pitch_joint">
+                <command_interface name="position">
+                    <param name="min">0</param>
+                    <param name="max">180</param>
+                </command_interface>
+                <state_interface name="position" />
+            </joint>
+            <joint name="right_ear_rotator_joint">
                 <command_interface name="position">
                     <param name="min">0</param>

File: ros_ws/src/bearmax_description/urdf/robot.urdf.xacro (robot description, xacro)
@@ -5,3 +5,11 @@
     <xacro:include filename="bearmax_description.urdf.xacro" />
     <xacro:include filename="hardware.ros2_control.xacro" />
+    <!--
+    <xacro:if value="$(arg use_ros2_control)">
+        <xacro:include filename="hardware.ros2_control.xacro" />
+    </xacro:if>
+    <xacro:unless value="$(arg use_ros2_control)">
+        <xacro:include filename="hardware.gazebo_control.xacro" />
+    </xacro:unless>
+    -->
 </robot>

Commit message: finished hardware interface for controller board communication and finalized bearmax urdf

File: ros_ws/src/bearmax_description/urdf/bearmax_description.urdf.xacro (robot description, xacro)
@@ -26,9 +26,9 @@
         />
       </geometry>
-      <!--material
+      <material
         name="">
         <color
           rgba="0.79216 0.81961 0.93333 1" />
-      </material-->
+      </material>
     </visual>
     <!--visual>
@@ -365,4 +365,15 @@
       velocity="100" />
   </joint>
+  <link name="left_arm_end_link">
+  </link>
+  <joint
+      name="left_arm_end_joint"
+      type="fixed">
+    <origin
+        xyz="0.1 0.0125 0"
+    />
+    <parent link="left_arm_elbow_link" />
+    <child link="left_arm_end_link" />
+  </joint>
   <link
     name="right_arm_shoulder_link">
@@ -543,4 +554,15 @@
       velocity="100" />
   </joint>
+  <link name="right_arm_end_link">
+  </link>
+  <joint
+      name="right_arm_end_joint"
+      type="fixed">
+    <origin
+        xyz="0.1 0.0075 0"
+    />
+    <parent link="right_arm_elbow_link" />
+    <child link="right_arm_end_link" />
+  </joint>
   <link
     name="head_platform_link">

File: ros_ws/src/bearmax_description/urdf/hardware.ros2_control.xacro (robot description, xacro)
@@ -1,3 +1,3 @@
-<?xml version="180.0"?>
+<?xml version="1.0"?>
 <robot xmlns:xacro="http://www.ros.org/wiki/xacro">
     <xacro:unless value="$(arg sim_mode)">
@@ -5,5 +5,5 @@
             <hardware>
                 <plugin>bearmax_hardware/BearmaxArduino</plugin>
-                <param name="device">/dev/ttyACM0</param>
+                <param name="device">/dev/pts/10</param>
                 <param name="baud_rate">57600</param>
                 <param name="timeout">180000</param>
@@ -62,5 +62,5 @@
                 <state_interface name="position" />
             </joint>
-            <joint name="right_ear_pitch">
+            <joint name="right_ear_pitch_joint">
                 <command_interface name="position">
                     <param name="min">0</param>

Commit message: Initial tasks and face following

File: ros_ws/src/bearmax_description/urdf/bearmax_description.urdf.xacro (robot description, xacro)
@@ -942,5 +942,5 @@
 	<parent link="camera_link"/>
 	<child link="camera_optical_link"/>
-	<origin xyz="0 0 0" rpy="${-pi/2} 0 ${-pi/2}"/>
+    <origin xyz="0 0 0" rpy="${-pi/2} 0 0"/>
   </joint>
 </robot>

File: ros_ws/src/bearmax_moveit_config/config/robot.ros2_control.xacro (robot description, xacro)
@@ -10,5 +10,4 @@
                 -->
                 <plugin>bearmax_hardware/BearmaxArduino</plugin>
-                <!-- Using /dev/pts/7 in place of actual serial port -->
                 <param name="device">/dev/ttyACM0</param>
                 <param name="baud_rate">57600</param>
